File: addon-microphone.kicad_sch (KiCad schematic)
At the start: 3 parts, among them J1 Conn_02x18_Odd_Even, J2 Conn_01x06, J3 Conn_01x06

Commit message: Add I2C EEPROM
Parts:
- added C1: 100n, Capacitor_THT:C_Disc_D5.0mm_W2.5mm_P5.00mm, symbol Device:C
- added JP1: Jumper_2_Open, Jumper:SolderJumper-2_P1.3mm_Open_RoundedPad1.0x1.5mm, symbol Jumper:Jumper_2_Open
- added R1: 1M, Resistor_THT:R_Axial_DIN0204_L3.6mm_D1.6mm_P7.62mm_Horizontal, symbol Device:R
- added U1: 24C02Cx-x-SN, Package_DIP:DIP-8_W7.62mm, symbol Memory_EEPROM:24C02Cx-x-SN
Connections:
- net +3.3V: now also C1.1, JP1.2 (B), U1.8 (VCC)
- net GND: now also C1.2, R1.1, U1.1 (A0), U1.2 (A1), U1.3 (A2), U1.4 (GND)
- net I2C_SDA: now reaches J1.10 (Pin_10)
- net I2C_SDA: now also U1.5 (SDA)
- net I2C_SCK: now reaches J1.9 (Pin_9)
- net I2C_SCK: now also U1.6 (SCL)
- new net: JP1.1 (A), R1.2, U1.7 (WP)
- no-connect marks 31 -> 29
Other:
- note added: "EEPRON Write protect"

Commit message: BF
Other:
- note added: "EEPROM Write protect"
- note removed: "EEPRON Write protect"
Changed lines of the file:
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@@
 		)
 	)
-	(text "EEPRON\nWrite\nprotect"
+	(text "EEPROM\nWrite\nprotect"
 		(exclude_from_sim no)
 		(at 198.374 91.948 0)
